Commit message: add hardware option for isaac

File: dual_arm_panda_moveit_config/config/panda.ros2_control.xacro (robot description, xacro)
@@ -1,9 +1,16 @@
 <?xml version="1.0"?>
 <robot xmlns:xacro="http://www.ros.org/wiki/xacro">
-    <xacro:macro name="panda_arm_ros2_control" params="name initial_positions_file prefix">
+    <xacro:macro name="panda_arm_ros2_control" params="name initial_positions_file prefix ros2_control_hardware_type">
         <xacro:property name="initial_positions" value="${xacro.load_yaml(initial_positions_file)['initial_positions']}"/>
-        <ros2_control name="${prefix}${name}" type="system">
+        <ros2_control name="${name}" type="system">
             <hardware>
-                <plugin>mock_components/GenericSystem</plugin>
+                <xacro:if value="${ros2_control_hardware_type == 'mock_components'}">
+                    <plugin>mock_components/GenericSystem</plugin>
+                </xacro:if>
+                <xacro:if value="${ros2_control_hardware_type == 'isaac'}">
+                    <plugin>topic_based_ros2_control/TopicBasedSystem</plugin>
+                    <param name="joint_commands_topic">/${prefix}isaac_joint_commands</param>
+                    <param name="joint_states_topic">/${prefix}isaac_joint_states</param>
+                </xacro:if>
             </hardware>
             <joint name="${prefix}panda_joint1">

File: dual_arm_panda_moveit_config/config/panda.urdf.xacro (robot description, xacro)
@@ -5,4 +5,5 @@
     <xacro:arg name="right_initial_positions_file"
             default="$(find dual_arm_panda_moveit_config)/config/right_initial_positions.yaml"/>
+    <xacro:arg name="ros2_control_hardware_type" default="mock_components" />
     <!-- Xacro imports -->
     <xacro:include filename="panda_arm_macro.xacro" />
@@ -42,5 +43,6 @@
         prefix="left_"
         parent="base"
-        initial_positions_file="$(arg left_initial_positions_file)">
+        initial_positions_file="$(arg left_initial_positions_file)"
+        ros2_control_hardware_type="$(arg ros2_control_hardware_type)">
         <origin xyz="0 -0.281 1" rpy="0 0 0" />
     </xacro:panda_arm>
@@ -50,5 +52,6 @@
         prefix="right_"
         parent="base"
-        initial_positions_file="$(arg right_initial_positions_file)">
+        initial_positions_file="$(arg right_initial_positions_file)"
+        ros2_control_hardware_type="$(arg ros2_control_hardware_type)">
         <origin xyz="0 0.281 1" rpy="0 0 0" />
     </xacro:panda_arm>

File: dual_arm_panda_moveit_config/config/panda_arm_macro.xacro (robot description, xacro)
@@ -1,10 +1,10 @@
 <?xml version="1.0" ?>
 <robot xmlns:xacro="http://www.ros.org/wiki/xacro">
-    <xacro:macro name="panda_arm" params="name prefix parent *origin initial_positions_file" >
+    <xacro:macro name="panda_arm" params="name prefix parent *origin initial_positions_file ros2_control_hardware_type" >
         <!-- ros2_control -->
         <xacro:include filename="$(find dual_arm_panda_moveit_config)/config/panda.ros2_control.xacro" />
-        <xacro:panda_arm_ros2_control name="${name}" initial_positions_file="${initial_positions_file}" prefix="${prefix}"/>
+        <xacro:panda_arm_ros2_control name="${name}_arm" initial_positions_file="${initial_positions_file}" prefix="${prefix}" ros2_control_hardware_type="${ros2_control_hardware_type}"/>
         <xacro:include filename="panda_hand.ros2_control.xacro" />
-        <xacro:panda_hand_ros2_control name="${name}" prefix="${prefix}"/>
+        <xacro:panda_hand_ros2_control name="${name}_hand" prefix="${prefix}" ros2_control_hardware_type="${ros2_control_hardware_type}"/>
         <!-- base_joint fixes base_link to the environment -->
         <joint name="${prefix}base_joint" type="fixed">

File: dual_arm_panda_moveit_config/config/panda_hand.ros2_control.xacro (robot description, xacro)
@@ -1,8 +1,15 @@
 <?xml version="1.0"?>
 <robot xmlns:xacro="http://www.ros.org/wiki/xacro">
-    <xacro:macro name="panda_hand_ros2_control" params="name prefix">
+    <xacro:macro name="panda_hand_ros2_control" params="name prefix ros2_control_hardware_type">
         <ros2_control name="${name}" type="system">
             <hardware>
-                <plugin>mock_components/GenericSystem</plugin>
+                <xacro:if value="${ros2_control_hardware_type == 'mock_components'}">
+                    <plugin>mock_components/GenericSystem</plugin>
+                </xacro:if>
+                <xacro:if value="${ros2_control_hardware_type == 'isaac'}">
+                    <plugin>topic_based_ros2_control/TopicBasedSystem</plugin>
+                    <param name="joint_commands_topic">/${prefix}isaac_joint_commands</param>
+                    <param name="joint_states_topic">/${prefix}isaac_joint_states</param>
+                </xacro:if>
             </hardware>
             <joint name="${prefix}panda_finger_joint1">
