Commit message: add small base for each robot

File: dual_arm_panda_moveit_config/config/panda_macro.srdf.xacro (robot description, xacro)
@@ -85,4 +85,22 @@
     <joint name="right_panda_joint7" value="1.5131"/>
   </group_state>
+   <group_state group="left_panda_arm" name="automatica_home">
+    <joint name="left_panda_joint1" value="-0.21829973"/>
+    <joint name="left_panda_joint2" value="0.1487587"/>
+    <joint name="left_panda_joint3" value="-0.06107414"/>
+    <joint name="left_panda_joint4" value="-2.20726548"/>
+    <joint name="left_panda_joint5" value="0.46944836"/>
+    <joint name="left_panda_joint6" value="2.21991352"/>
+    <joint name="left_panda_joint7" value="-1.3412202"/>
+  </group_state>
+  <group_state group="right_panda_arm" name="automatica_home">
+    <joint name="right_panda_joint1" value="-0.66797274"/>
+    <joint name="right_panda_joint2" value="0.6828252"/>
+    <joint name="right_panda_joint3" value="-0.18094061"/>
+    <joint name="right_panda_joint4" value="-1.31640549"/>
+    <joint name="right_panda_joint5" value="0.06258675"/>
+    <joint name="right_panda_joint6" value="2.04563806"/>
+    <joint name="right_panda_joint7" value="-1.62984602"/>
+  </group_state>
   <group_state group="left_hand" name="open">
     <joint name="left_panda_finger_joint1" value="0.035"/>
@@ -107,4 +125,6 @@
   <!--VIRTUAL JOINT: Purpose: this element defines a virtual joint between a robot link and an external frame of reference (considered fixed with respect to the robot)-->
   <virtual_joint name="virtual_joint" type="fixed" parent_frame="world" child_link="base"/>
+  <virtual_joint name="virtual_joint" type="fixed" parent_frame="base" child_link="left_base"/>
+  <virtual_joint name="virtual_joint" type="fixed" parent_frame="base" child_link="right_base"/>
   <!-- <virtual_joint name="virtual_joint_1" type="fixed" parent_frame="base" child_link="left_panda_link0"/>
   <virtual_joint name="virtual_joint_2" type="fixed" parent_frame="base" child_link="right_panda_link0"/> -->
@@ -115,4 +135,11 @@
   <disable_collisions link1="base" link2="left_panda_link3" reason="Never"/>
   <disable_collisions link1="base" link2="left_panda_link4" reason="Never"/>
+  <disable_collisions link1="base" link2="left_base" reason="Adjacent"/>
+  <disable_collisions link1="left_base" link2="left_panda_link0" reason="Adjacent"/>
+  <disable_collisions link1="left_base" link2="left_panda_link1" reason="Default"/>
+  <disable_collisions link1="left_base" link2="left_panda_link2" reason="Never"/>
+  <disable_collisions link1="left_base" link2="left_panda_link3" reason="Never"/>
+  <disable_collisions link1="left_base" link2="left_panda_link4" reason="Never"/>
+  <disable_collisions link1="left_base" link2="right_base" reason="Never"/>
   <disable_collisions link1="base" link2="right_panda_link0" reason="Adjacent"/>
   <disable_collisions link1="base" link2="right_panda_link1" reason="Default"/>
@@ -120,4 +147,10 @@
   <disable_collisions link1="base" link2="right_panda_link3" reason="Never"/>
   <disable_collisions link1="base" link2="right_panda_link4" reason="Never"/>
+  <disable_collisions link1="base" link2="right_base" reason="Adjacent"/>
+  <disable_collisions link1="right_base" link2="right_panda_link0" reason="Adjacent"/>
+  <disable_collisions link1="right_base" link2="right_panda_link1" reason="Default"/>
+  <disable_collisions link1="right_base" link2="right_panda_link2" reason="Never"/>
+  <disable_collisions link1="right_base" link2="right_panda_link3" reason="Never"/>
+  <disable_collisions link1="right_base" link2="right_panda_link4" reason="Never"/>
   <disable_collisions link1="left_panda_link0" link2="left_panda_link1" reason="Adjacent"/>
   <disable_collisions link1="left_panda_link0" link2="left_panda_link2" reason="Never"/>
