Commit message: add base and change positions in dual setup

File: dual_arm_panda_moveit_config/config/panda.urdf.xacro (robot description, xacro)
@@ -8,5 +8,33 @@
     <link name="world"/>
     <!-- Xacro imports -->
-    <xacro:include filename="panda_arm_macro.xacro" />
+    <xacro:include filename="panda_arm_macro.xacro" />\
+    <!-- box shaped table as base for the 2 Pandas -->
+    <link name="base">
+        <visual>
+        <origin xyz="0.09 0 0.5" rpy="0 0 0" />
+        <geometry>
+            <box size="0.8 1.6 1" />
+        </geometry>
+        <material name="White">
+            <color rgba="1.0 1.0 1.0 1.0" />
+        </material>
+        </visual>
+        <collision>
+        <origin xyz="0.09 0 0.5" rpy="0 0 0" />
+        <geometry>
+            <box size="0.8 1.6 1" />
+        </geometry>
+        </collision>
+        <inertial>
+        <origin xyz="0.0 0.0 0.0" rpy="0.0 0.0 0.0"/>
+        <mass value="10.0"/>
+        <inertia ixx="0.001" ixy="0.0" ixz="0.001" iyy="0.0" iyz="0.0" izz="0.001"/>
+        </inertial>
+    </link>
+    <joint name="base_to_world" type="fixed">
+            <parent link="world"/>
+            <child link="base"/>
+            <origin xyz="0.0 0.0 0.0" rpy="0.0 0.0 0.0"/>
+    </joint>
     <!-- Left arm -->
     <xacro:panda_arm
@@ -15,5 +43,5 @@
         parent="world"
         initial_positions_file="$(arg left_initial_positions_file)">
-        <origin xyz="0 -1.5 0" rpy="0 0 0" />
+        <origin xyz="0 -0.281 1" rpy="0 0 0" />
     </xacro:panda_arm>
     <!-- Right arm -->
@@ -23,5 +51,5 @@
         parent="world"
         initial_positions_file="$(arg right_initial_positions_file)">
-        <origin xyz="0 1.5 0" rpy="0 0 0" />
+        <origin xyz="0 0.281 1" rpy="0 0 0" />
     </xacro:panda_arm>
 </robot>

Commit message: add senseone option in urdf

File: dual_arm_panda_moveit_config/config/panda.urdf.xacro (robot description, xacro)
@@ -6,6 +6,9 @@
             default="$(find dual_arm_panda_moveit_config)/config/right_initial_positions.yaml"/>
     <xacro:arg name="ros2_control_hardware_type" default="mock_components" />
+    <xacro:arg name="use_sensone_left" default="false" />
+    <xacro:arg name="use_sensone_right" default="false" />
     <!-- Xacro imports -->
     <xacro:include filename="panda_arm_macro.xacro" />
+    <xacro:include filename="panda_arm_sensone_macro.xacro" />
     <!-- Root link -->
     <link name="world"/>
@@ -39,20 +42,44 @@
     </joint>
     <!-- Left arm -->
-    <xacro:panda_arm
-        name="left_panda"
-        prefix="left_"
-        parent="base"
-        initial_positions_file="$(arg left_initial_positions_file)"
-        ros2_control_hardware_type="$(arg ros2_control_hardware_type)">
-        <origin xyz="0 -0.281 1" rpy="0 0 0" />
-    </xacro:panda_arm>
+    <xacro:if value="$(arg use_sensone_left)">
+        <xacro:panda_arm_sensone
+            name="left_panda"
+            prefix="left_"
+            parent="base"
+            initial_positions_file="$(arg left_initial_positions_file)"
+            ros2_control_hardware_type="$(arg ros2_control_hardware_type)">
+            <origin xyz="0 -0.281 1" rpy="0 0 0" />
+        </xacro:panda_arm_sensone>
+    </xacro:if>
+    <xacro:unless value="$(arg use_sensone_left)">
+        <xacro:panda_arm
+            name="left_panda"
+            prefix="left_"
+            parent="base"
+            initial_positions_file="$(arg left_initial_positions_file)"
+            ros2_control_hardware_type="$(arg ros2_control_hardware_type)">
+            <origin xyz="0 -0.281 1" rpy="0 0 0" />
+        </xacro:panda_arm>
+    </xacro:unless>
     <!-- Right arm -->
-    <xacro:panda_arm
-        name="right_panda"
-        prefix="right_"
-        parent="base"
-        initial_positions_file="$(arg right_initial_positions_file)"
-        ros2_control_hardware_type="$(arg ros2_control_hardware_type)">
-        <origin xyz="0 0.281 1" rpy="0 0 0" />
-    </xacro:panda_arm>
+    <xacro:if value="$(arg use_sensone_right)">
+        <xacro:panda_arm_sensone
+            name="right_panda"
+            prefix="right_"
+            parent="base"
+            initial_positions_file="$(arg right_initial_positions_file)"
+            ros2_control_hardware_type="$(arg ros2_control_hardware_type)">
+            <origin xyz="0 0.281 1" rpy="0 0 0" />
+        </xacro:panda_arm_sensone>
+    </xacro:if>
+    <xacro:unless value="$(arg use_sensone_right)">
+        <xacro:panda_arm
+            name="right_panda"
+            prefix="right_"
+            parent="base"
+            initial_positions_file="$(arg right_initial_positions_file)"
+            ros2_control_hardware_type="$(arg ros2_control_hardware_type)">
+            <origin xyz="0 0.281 1" rpy="0 0 0" />
+        </xacro:panda_arm>
+    </xacro:unless>
 </robot>

Commit message: add small base for each robot

File: dual_arm_panda_moveit_config/config/panda.urdf.xacro (robot description, xacro)
@@ -37,9 +37,37 @@
     </link>
     <joint name="base_to_world" type="fixed">
-            <parent link="world"/>
-            <child link="base"/>
-            <origin xyz="0.0 0.0 0.0" rpy="0.0 0.0 0.0"/>
+        <parent link="world"/>
+        <child link="base"/>
+        <origin xyz="0.0 0.0 0.0" rpy="0.0 0.0 0.0"/>
     </joint>
     <!-- Left arm -->
+    <!-- left arm base -->
+    <link name="left_base">
+        <visual>
+        <origin xyz="-0.055 -0.281 1.0125" rpy="0 0 0" />
+        <geometry>
+            <box size="0.25 0.25 0.025" />
+        </geometry>
+        <material name="White">
+            <color rgba="1.0 1.0 1.0 1.0" />
+        </material>
+        </visual>
+        <collision>
+        <origin xyz="0.09 0 0.5" rpy="0 0 0" />
+        <geometry>
+            <box size="0.8 1.6 1" />
+        </geometry>
+        </collision>
+        <inertial>
+        <origin xyz="0.0 0.0 0.0" rpy="0.0 0.0 0.0"/>
+        <mass value="10.0"/>
+        <inertia ixx="0.001" ixy="0.0" ixz="0.001" iyy="0.0" iyz="0.0" izz="0.001"/>
+        </inertial>
+    </link>
+    <joint name="left_base_to_world" type="fixed">
+        <parent link="base"/>
+        <child link="left_base"/>
+        <origin xyz="0.0 0.0 0.0" rpy="0.0 0.0 0.0"/>
+    </joint>
     <xacro:if value="$(arg use_sensone_left)">
         <xacro:panda_arm_sensone
@@ -49,5 +77,5 @@
             initial_positions_file="$(arg left_initial_positions_file)"
             ros2_control_hardware_type="$(arg ros2_control_hardware_type)">
-            <origin xyz="0 -0.281 1" rpy="0 0 0" />
+            <origin xyz="0 -0.281 1.025" rpy="0 0 0" />
         </xacro:panda_arm_sensone>
     </xacro:if>
@@ -59,8 +87,36 @@
             initial_positions_file="$(arg left_initial_positions_file)"
             ros2_control_hardware_type="$(arg ros2_control_hardware_type)">
-            <origin xyz="0 -0.281 1" rpy="0 0 0" />
+            <origin xyz="0 -0.281 1.025" rpy="0 0 0" />
         </xacro:panda_arm>
     </xacro:unless>
     <!-- Right arm -->
+    <!-- right arm base -->
+    <link name="right_base">
+        <visual>
+        <origin xyz="-0.055 0.281 1.0125" rpy="0 0 0" />
+        <geometry>
+            <box size="0.25 0.25 0.025" />
+        </geometry>
+        <material name="White">
+            <color rgba="1.0 1.0 1.0 1.0" />
+        </material>
+        </visual>
+        <collision>
+        <origin xyz="0.09 0 0.5" rpy="0 0 0" />
+        <geometry>
+            <box size="0.8 1.6 1" />
+        </geometry>
+        </collision>
+        <inertial>
+        <origin xyz="0.0 0.0 0.0" rpy="0.0 0.0 0.0"/>
+        <mass value="10.0"/>
+        <inertia ixx="0.001" ixy="0.0" ixz="0.001" iyy="0.0" iyz="0.0" izz="0.001"/>
+        </inertial>
+    </link>
+    <joint name="right_base_to_world" type="fixed">
+        <parent link="base"/>
+        <child link="right_base"/>
+        <origin xyz="0.0 0.0 0.0" rpy="0.0 0.0 0.0"/>
+    </joint>
     <xacro:if value="$(arg use_sensone_right)">
         <xacro:panda_arm_sensone
@@ -70,5 +126,5 @@
             initial_positions_file="$(arg right_initial_positions_file)"
             ros2_control_hardware_type="$(arg ros2_control_hardware_type)">
-            <origin xyz="0 0.281 1" rpy="0 0 0" />
+            <origin xyz="0 0.281 1.025" rpy="0 0 0" />
         </xacro:panda_arm_sensone>
     </xacro:if>
@@ -80,5 +136,5 @@
             initial_positions_file="$(arg right_initial_positions_file)"
             ros2_control_hardware_type="$(arg ros2_control_hardware_type)">
-            <origin xyz="0 0.281 1" rpy="0 0 0" />
+            <origin xyz="0 0.281 1.025" rpy="0 0 0" />
         </xacro:panda_arm>
     </xacro:unless>

Commit message: align world origin to center of robot base

File: dual_arm_panda_moveit_config/config/panda.urdf.xacro (robot description, xacro)
@@ -16,5 +16,5 @@
     <link name="base">
         <visual>
-        <origin xyz="0.09 0 0.5" rpy="0 0 0" />
+        <origin xyz="0.09 0 -0.525" rpy="0 0 0" />
         <geometry>
             <box size="0.8 1.6 1" />
@@ -25,5 +25,5 @@
         </visual>
         <collision>
-        <origin xyz="0.09 0 0.5" rpy="0 0 0" />
+        <origin xyz="0.09 0 -0.525" rpy="0 0 0" />
         <geometry>
             <box size="0.8 1.6 1" />
@@ -45,5 +45,5 @@
     <link name="left_base">
         <visual>
-        <origin xyz="-0.055 -0.281 1.0125" rpy="0 0 0" />
+        <origin xyz="-0.04 -0.281 -0.0125" rpy="0 0 0" />
         <geometry>
             <box size="0.25 0.25 0.025" />
@@ -53,10 +53,10 @@
         </material>
         </visual>
-        <collision>
+        <!-- <collision>
         <origin xyz="0.09 0 0.5" rpy="0 0 0" />
         <geometry>
             <box size="0.8 1.6 1" />
         </geometry>
-        </collision>
+        </collision> -->
         <inertial>
         <origin xyz="0.0 0.0 0.0" rpy="0.0 0.0 0.0"/>
@@ -77,5 +77,5 @@
             initial_positions_file="$(arg left_initial_positions_file)"
             ros2_control_hardware_type="$(arg ros2_control_hardware_type)">
-            <origin xyz="0 -0.281 1.025" rpy="0 0 0" />
+            <origin xyz="0 -0.281 0.0" rpy="0 0 0" />
         </xacro:panda_arm_sensone>
     </xacro:if>
@@ -87,5 +87,5 @@
             initial_positions_file="$(arg left_initial_positions_file)"
             ros2_control_hardware_type="$(arg ros2_control_hardware_type)">
-            <origin xyz="0 -0.281 1.025" rpy="0 0 0" />
+            <origin xyz="0 -0.281 0.0" rpy="0 0 0" />
         </xacro:panda_arm>
     </xacro:unless>
@@ -94,5 +94,5 @@
     <link name="right_base">
         <visual>
-        <origin xyz="-0.055 0.281 1.0125" rpy="0 0 0" />
+        <origin xyz="-0.04 0.281 -0.0125" rpy="0 0 0" />
         <geometry>
             <box size="0.25 0.25 0.025" />
@@ -102,10 +102,10 @@
         </material>
         </visual>
-        <collision>
-        <origin xyz="0.09 0 0.5" rpy="0 0 0" />
+        <!-- <collision>
+        <origin xyz="-0.04 0.281 -0.0125" rpy="0 0 0" />
         <geometry>
             <box size="0.8 1.6 1" />
         </geometry>
-        </collision>
+        </collision> -->
         <inertial>
         <origin xyz="0.0 0.0 0.0" rpy="0.0 0.0 0.0"/>
@@ -126,5 +126,5 @@
             initial_positions_file="$(arg right_initial_positions_file)"
             ros2_control_hardware_type="$(arg ros2_control_hardware_type)">
-            <origin xyz="0 0.281 1.025" rpy="0 0 0" />
+            <origin xyz="0 0.281 0.0" rpy="0 0 0" />
         </xacro:panda_arm_sensone>
     </xacro:if>
@@ -136,5 +136,5 @@
             initial_positions_file="$(arg right_initial_positions_file)"
             ros2_control_hardware_type="$(arg ros2_control_hardware_type)">
-            <origin xyz="0 0.281 1.025" rpy="0 0 0" />
+            <origin xyz="0 0.281 0.0" rpy="0 0 0" />
         </xacro:panda_arm>
     </xacro:unless>

Commit message: add alter finger

File: dual_arm_panda_moveit_config/config/panda.urdf.xacro (robot description, xacro)
@@ -7,8 +7,11 @@
     <xacro:arg name="ros2_control_hardware_type" default="mock_components" />
     <xacro:arg name="use_sensone_left" default="false" />
+    <xacro:arg name="alter_finger_left" default="false" />
     <xacro:arg name="use_sensone_right" default="false" />
+    <xacro:arg name="alter_finger_right" default="false" />
     <!-- Xacro imports -->
     <xacro:include filename="panda_arm_macro.xacro" />
     <xacro:include filename="panda_arm_sensone_macro.xacro" />
+    <xacro:include filename="panda_arm_alter_finger_macro.xacro" />
     <!-- Root link -->
     <link name="world"/>
@@ -81,4 +84,15 @@
     </xacro:if>
     <xacro:unless value="$(arg use_sensone_left)">
+        <xacro:if value="$(arg alter_finger_left)">
+            <xacro:panda_arm_alter_finger
+                name="left_panda"
+                prefix="left_"
+                parent="base"
+                initial_positions_file="$(arg left_initial_positions_file)"
+                ros2_control_hardware_type="$(arg ros2_control_hardware_type)">
+                <origin xyz="0 -0.281 0.0" rpy="0 0 0" />
+            </xacro:panda_arm_alter_finger>
+        </xacro:if>
+        <xacro:unless value="$(arg alter_finger_left)">
         <xacro:panda_arm
             name="left_panda"
@@ -89,4 +103,5 @@
             <origin xyz="0 -0.281 0.0" rpy="0 0 0" />
         </xacro:panda_arm>
+        </xacro:unless>
     </xacro:unless>
     <!-- Right arm -->
@@ -130,4 +145,15 @@
     </xacro:if>
     <xacro:unless value="$(arg use_sensone_right)">
+        <xacro:if value="$(arg alter_finger_right)">
+            <xacro:panda_arm_alter_finger
+                name="right_panda"
+                prefix="right_"
+                parent="base"
+                initial_positions_file="$(arg right_initial_positions_file)"
+                ros2_control_hardware_type="$(arg ros2_control_hardware_type)">
+                <origin xyz="0 0.281 0.0" rpy="0 0 0" />
+            </xacro:panda_arm_alter_finger>
+        </xacro:if>
+        <xacro:unless value="$(arg alter_finger_right)">
         <xacro:panda_arm
             name="right_panda"
@@ -138,4 +164,5 @@
             <origin xyz="0 0.281 0.0" rpy="0 0 0" />
         </xacro:panda_arm>
+        </xacro:unless>
     </xacro:unless>
 </robot>
